Commit message: changes to get gazebo sim working

File: ur_description/urdf/inc/ur_macro_bb.xacro (robot description, xacro)
@@ -321,5 +321,5 @@
         <origin rpy="1.57079632679 0 0.0" xyz="0 0 0"/>
         <child link="wrist_3_old"/>
-        <parent link="wrist_3_link"/>
+        <parent link="${prefix}wrist_3_link"/>
     </joint>
     <link name="wrist_3_old"></link>
@@ -346,5 +346,6 @@
         </collision>
         <inertial>
-            <mass value="0.5"/>
+            <!-- <mass value="0.5"/> -->
+            <mass value="0.1"/>
             <origin rpy=" 0 0 0" xyz="0.0 0 0.0"/>
             <inertia ixx="1.0" ixy="0" ixz="0" iyy="1.0" iyz="0" izz="1.0"/>
@@ -357,4 +358,5 @@
     </joint>
     <!-- I am not sure why both this and ee_link (can remove ee_link) but leaving for now-->
+    <!-- Actually looks like ee_link is used by gazebo, so inhand_link would be one to remove, but it's needed for mesh.-->
     <link name="inhand_link">
         <visual>
@@ -374,5 +376,5 @@
         </collision>
         <inertial>
-            <mass value="0.2"/>
+            <mass value="0.1"/>
             <origin rpy=" 0 0 0" xyz="0.08 0.084 0.07"/>
             <inertia ixx="1.0" ixy="0" ixz="0" iyy="1.0" iyz="0" izz="1.0"/>

File: ur_gazebo/urdf/ur.xacro (robot description, xacro)
@@ -65,5 +65,5 @@
     <parent link="world"/>
     <child link="base_link"/>
-    <origin xyz="0 0 0" rpy="0 0 0"/>
+    <origin xyz="0.0 0.0 1.54" rpy="1.5707 0.0 1.5707"/>
   </joint>
   <link name="tool0_controller"/>

File: ur_gazebo/urdf/ur_macro.xacro (robot description, xacro)
@@ -46,5 +46,6 @@
       the definitions for the real robot.
     -->
-  <xacro:include filename="$(find ur_description)/urdf/inc/ur_macro.xacro"/>
+  <xacro:include filename="$(find ur_description)/urdf/inc/ur_macro_bb.xacro"/>
+  <!-- <xacro:include filename="$(find ur_description)/urdf/inc/ur_macro.xacro"/> -->
     <!-- Instantiate model for the REAL robot. -->
     <xacro:ur_robot

Commit message: real robot moving

File: ur_description/urdf/inc/ur_macro_bb.xacro (robot description, xacro)
@@ -349,5 +349,6 @@
             <mass value="0.1"/>
             <origin rpy=" 0 0 0" xyz="0.0 0 0.0"/>
-            <inertia ixx="1.0" ixy="0" ixz="0" iyy="1.0" iyz="0" izz="1.0"/>
+            <!-- <inertia ixx="1.0" ixy="0" ixz="0" iyy="1.0" iyz="0" izz="1.0"/> -->
+            <inertia ixx="0.01" ixy="0" ixz="0" iyy="0.01" iyz="0" izz="0.01"/>
         </inertial>
     </link>
@@ -378,5 +379,6 @@
             <mass value="0.1"/>
             <origin rpy=" 0 0 0" xyz="0.08 0.084 0.07"/>
-            <inertia ixx="1.0" ixy="0" ixz="0" iyy="1.0" iyz="0" izz="1.0"/>
+            <!-- <inertia ixx="1.0" ixy="0" ixz="0" iyy="1.0" iyz="0" izz="1.0"/> -->
+            <inertia ixx="0.01" ixy="0" ixz="0" iyy="0.01" iyz="0" izz="0.01"/>
         </inertial>
     </link>

File: ur_description/urdf/ur.xacro (robot description, xacro)
@@ -29,3 +29,10 @@
      safety_pos_margin="$(arg safety_pos_margin)"
      safety_k_position="$(arg safety_k_position)"/>
+      <!-- Harry added this to fix setJointLimits bug -->
+      <link name="world"/>
+      <joint name="world_joint" type="fixed">
+            <parent link="world"/>
+            <child link="base_link"/>
+            <origin xyz="0.0 0.0 1.54" rpy="1.5707 0.0 1.5707"/>
+      </joint>
 </robot>

Commit message: reduce inertia, add stereo camera

File: ur_description/urdf/inc/ur_macro_bb.xacro (robot description, xacro)
@@ -350,5 +350,5 @@
             <origin rpy=" 0 0 0" xyz="0.0 0 0.0"/>
             <!-- <inertia ixx="1.0" ixy="0" ixz="0" iyy="1.0" iyz="0" izz="1.0"/> -->
-            <inertia ixx="0.01" ixy="0" ixz="0" iyy="0.01" iyz="0" izz="0.01"/>
+            <inertia ixx="0.001" ixy="0" ixz="0" iyy="0.001" iyz="0" izz="0.001"/>
         </inertial>
     </link>
@@ -380,5 +380,5 @@
             <origin rpy=" 0 0 0" xyz="0.08 0.084 0.07"/>
             <!-- <inertia ixx="1.0" ixy="0" ixz="0" iyy="1.0" iyz="0" izz="1.0"/> -->
-            <inertia ixx="0.01" ixy="0" ixz="0" iyy="0.01" iyz="0" izz="0.01"/>
+            <inertia ixx="0.001" ixy="0" ixz="0" iyy="0.001" iyz="0" izz="0.001"/>
         </inertial>
     </link>
@@ -398,5 +398,5 @@
     <joint name="ee_link_to_inhand_cam_link" type="fixed">
         <origin xyz="0 0 0" rpy="${-pi/2} 0 ${-pi/2} "/>
-        <parent link="ee_link"/>
+        <parent link="${prefix}ee_link"/>
         <child link="inhand_cam_link"/>
     </joint>

File: ur_gazebo/urdf/ur_macro.xacro (robot description, xacro)
@@ -81,4 +81,57 @@
     <gazebo reference="${prefix}ee_link">
       <selfCollide>true</selfCollide>
+      <sensor type="multicamera" name="stereo_camera">
+        <update_rate>1.0</update_rate>
+        <camera name="left">
+          <pose>0 0 0 0 0 0</pose>
+          <horizontal_fov>0.777</horizontal_fov>
+          <image>
+            <width>1440</width>
+            <height>1080</height>
+            <format>R8G8B8</format>
+          </image>
+          <clip>
+            <near>0.02</near>
+            <far>300</far>
+          </clip>
+          <noise>
+            <type>gaussian</type>
+            <mean>0.0</mean>
+            <stddev>0.0</stddev>
+          </noise>
+        </camera>
+        <camera name="right">
+          <pose>0 -0.06 0 0 0 0</pose>
+          <horizontal_fov>0.777</horizontal_fov>
+          <image>
+            <width>1440</width>
+            <height>1080</height>
+            <format>R8G8B8</format>
+          </image>
+          <clip>
+            <near>0.02</near>
+            <far>300</far>
+          </clip>
+          <noise>
+            <type>gaussian</type>
+            <mean>0.0</mean>
+            <stddev>0.0</stddev>
+          </noise>
+        </camera>
+        <plugin name="stereo_camera_controller" filename="libgazebo_ros_multicamera.so">
+          <alwaysOn>true</alwaysOn>
+          <updateRate>0.0</updateRate>
+          <cameraName>theia</cameraName>
+          <imageTopicName>image_raw_sim</imageTopicName>
+          <cameraInfoTopicName>camera_info_sim</cameraInfoTopicName>
+          <frameName>camera</frameName>
+          <hackBaseline>0.06</hackBaseline>
+          <distortionK1>0.0</distortionK1>
+          <distortionK2>0.0</distortionK2>
+          <distortionK3>0.0</distortionK3>
+          <distortionT1>0.0</distortionT1>
+          <distortionT2>0.0</distortionT2>
+        </plugin>
+      </sensor>
     </gazebo>
     <!--

Commit message: remove inertia ee, reduce p in controller

File: ur_description/urdf/inc/ur_macro_bb.xacro (robot description, xacro)
@@ -345,11 +345,4 @@
             </geometry>
         </collision>
-        <inertial>
-            <!-- <mass value="0.5"/> -->
-            <mass value="0.1"/>
-            <origin rpy=" 0 0 0" xyz="0.0 0 0.0"/>
-            <!-- <inertia ixx="1.0" ixy="0" ixz="0" iyy="1.0" iyz="0" izz="1.0"/> -->
-            <inertia ixx="0.001" ixy="0" ixz="0" iyy="0.001" iyz="0" izz="0.001"/>
-        </inertial>
     </link>
     <joint name="ee_base_link_to_inhand_joint" type="fixed">
@@ -376,10 +369,4 @@
             </geometry>
         </collision>
-        <inertial>
-            <mass value="0.1"/>
-            <origin rpy=" 0 0 0" xyz="0.08 0.084 0.07"/>
-            <!-- <inertia ixx="1.0" ixy="0" ixz="0" iyy="1.0" iyz="0" izz="1.0"/> -->
-            <inertia ixx="0.001" ixy="0" ixz="0" iyy="0.001" iyz="0" izz="0.001"/>
-        </inertial>
     </link>
     <joint name="${prefix}ee_fixed_joint" type="fixed">
