Commit message: get to work with slider

File: ur_description/urdf/inc/ur_macro_bb_no_slider.xacro (robot description, xacro)
@@ -66,32 +66,22 @@
     <link name="${prefix}base_link"/>
     <link name="${prefix}base_link_inertia">
-      <inertial>
-        <mass value="1.0" />
-        <inertia ixx="1.0" ixy="0.0" ixz="0.0" iyy="1.0" iyz="0.0" izz="1.0" />
-      </inertial>
-      <visual>
-        <!-- <origin xyz="0 0 0" rpy="0 0 ${pi}"/> -->
-        <origin rpy="0 ${-1* pi / 2}  0" xyz="0 0 0"/>
-        <geometry>
-          <!-- <mesh filename="${base_visual_mesh}"/> -->
-          <mesh filename="package://ros_urdf_tutorial/slide_mesh/corrected/linear_slide_reduced_origin_fixed.stl" scale="0.001 0.001 0.001"/>
-        </geometry>
-        <!-- <material name="${base_visual_material_name}"> -->
-          <!-- <color rgba="${base_visual_material_color}"/> -->
-        <material name="LightGrey">
-          <color rgba="0.7 0.7 0.7 1.0"/>
-        </material>
-      </visual>
-      <collision>
-        <!-- <origin xyz="0 0 0" rpy="0 0 ${pi}"/> -->
-        <origin rpy="0 ${-1* pi / 2}  0" xyz="0 0 0"/>
-        <geometry>
-          <!-- <mesh filename="${base_collision_mesh}"/> -->
-          <mesh filename="package://ros_urdf_tutorial/slide_mesh/corrected/linear_slide_reduced_origin_fixed.stl" scale="0.001 0.001 0.001"/>
-        </geometry>
-      </collision>
-      <!-- <xacro:cylinder_inertial radius="${base_inertia_radius}" length="${base_inertia_length}" mass="${base_mass}">
+      <visual>
+        <origin xyz="0 0 0" rpy="0 0 ${pi}"/>
+        <geometry>
+          <mesh filename="${base_visual_mesh}"/>
+        </geometry>
+        <material name="${base_visual_material_name}">
+          <color rgba="${base_visual_material_color}"/>
+        </material>
+      </visual>
+      <collision>
+        <origin xyz="0 0 0" rpy="0 0 ${pi}"/>
+        <geometry>
+          <mesh filename="${base_collision_mesh}"/>
+        </geometry>
+      </collision>
+      <xacro:cylinder_inertial radius="${base_inertia_radius}" length="${base_inertia_length}" mass="${base_mass}">
         <origin xyz="0 0 0" rpy="0 0 0" />
-      </xacro:cylinder_inertial> -->
+      </xacro:cylinder_inertial>
     </link>
     <link name="${prefix}shoulder_link">
@@ -225,21 +215,10 @@
            link/frame) to introduce the necessary rotation over Z (of pi rad).
       -->
-      <!-- <origin xyz="0 0 0" rpy="0 0 ${pi}" /> -->
-      <origin xyz="0 0 0" rpy="0 0 0" />
-    </joint>
-    <!-- I added this here first so that it is first in list -->
-    <joint name="${prefix}sliding_base_joint" type="prismatic">
-		  <parent link="${prefix}base_link_inertia"/>
-		  <child link="${prefix}camera_link_"/>
-		  <limit effort="1" lower="-0.675" upper="0.675" velocity="0.25" acceleration="2.5"/>
-		  <axis xyz = "0 1 0"/>
-		  <origin xyz="0.0 0.0 0.0" rpy="0 0 0" />
-	  </joint>
+      <origin xyz="0 0 0" rpy="0 0 ${pi}" />
+    </joint>
     <joint name="${prefix}shoulder_pan_joint" type="revolute">
-      <!-- <parent link="${prefix}base_link_inertia" /> -->
-      <parent link="${prefix}ur_base_link" />
+      <parent link="${prefix}base_link_inertia" />
       <child link="${prefix}shoulder_link" />
-      <!-- <origin xyz="${shoulder_x} ${shoulder_y} ${shoulder_z}" rpy="${shoulder_roll} ${shoulder_pitch} ${shoulder_yaw}" /> -->
-      <origin xyz="0.0 0.0 0.089159" rpy="0.0 0.0 ${pi}" />
+      <origin xyz="${shoulder_x} ${shoulder_y} ${shoulder_z}" rpy="${shoulder_roll} ${shoulder_pitch} ${shoulder_yaw}" />
       <axis xyz="0 0 1" />
       <limit lower="${shoulder_pan_lower_limit}" upper="${shoulder_pan_upper_limit}"
@@ -411,50 +390,4 @@
     <link name="inhand_cam_link"></link>
     <!-- ======================== END-EFFECTOR END==========================-->
-    <!-- ======================== SLIDING-BASE START==========================-->
-    <link name="camera_link_">
-		  <visual>
-			  <geometry>
-				  <mesh filename="package://ros_urdf_tutorial/slide_mesh/corrected/camera_system_stl_reduced_origin_fixed.stl" scale="0.001 0.001 0.001"/>
-			  </geometry>
-			  <origin rpy="0 -1.5708 0" xyz="0 0 0.053012 "/>
-				<material name="white">
-			    <color rgba="1 1 1 1"/>
-			  </material>
-		  </visual>
-		  <collision>
-			  <geometry>
-				  <mesh filename="package://ros_urdf_tutorial/slide_mesh/corrected/camera_system_stl_reduced_origin_fixed.stl" scale="0.001 0.001 0.001"/>
-			  </geometry>
-			  <origin rpy="0 -1.5708 0" xyz="0 0 0.053012 "/>
-		  </collision>
-		  <inertial>
-			  <mass value="1"/>
-			  <inertia ixx="1.0" ixy="0.0" ixz="0.0" iyy="1.0" iyz="0.0" izz="1.0"/>
-		  </inertial>
-	  </link>
-    <joint name="camera_ur_base_joint" type="fixed">
-      <origin rpy="0 0 0" xyz="0 0 0.138352 "/>
-      <parent link="camera_link_"/>
-      <child link="ur_base_link"/>
-    </joint>
-    <link name="${prefix}ur_base_link" >
-      <visual>
-        <geometry>
-          <mesh filename="package://ur_description/meshes/ur5/visual/base.dae" />
-        </geometry>
-        <material name="LightGrey">
-          <color rgba="0.7 0.7 0.7 1.0"/>
-        </material>
-      </visual>
-      <collision>
-        <geometry>
-          <mesh filename="package://ur_description/meshes/ur5/collision/base.stl" />
-        </geometry>
-      </collision>
-      <xacro:cylinder_inertial radius="0.06" length="0.05" mass="${base_mass}">
-        <origin xyz="0.0 0.0 0.0" rpy="0 0 0" />
-      </xacro:cylinder_inertial>
-    </link>
-    <!-- ======================== SLIDING-BASE START==========================-->
   </xacro:macro>
 </robot>

File: ur_description/urdf/inc/ur_transmissions.xacro (robot description, xacro)
@@ -7,4 +7,14 @@
   -->
   <xacro:macro name="ur_arm_transmission" params="prefix hw_interface">
+    <!-- I added sliding base -->
+    <transmission name="${prefix}sliding_base_trans">
+      <type>transmission_interface/SimpleTransmission</type>
+      <joint name="${prefix}sliding_base_joint">
+        <hardwareInterface>${hw_interface}</hardwareInterface>
+      </joint>
+      <actuator name="${prefix}sliding_base_motor">
+        <mechanicalReduction>1</mechanicalReduction>
+      </actuator>
+    </transmission>
     <transmission name="${prefix}shoulder_pan_trans">
       <type>transmission_interface/SimpleTransmission</type>

File: ur_description/urdf/ur.xacro (robot description, xacro)
@@ -34,5 +34,8 @@
             <parent link="world"/>
             <child link="base_link"/>
+            <origin xyz="0.0 0.0 1.54" rpy="0.0 1.5707 0.0"/>
+            <!-- was this before sliding base added
             <origin xyz="0.0 0.0 1.54" rpy="1.5707 0.0 1.5707"/>
+            -->
       </joint>
 </robot>

File: ur_gazebo/urdf/ur.xacro (robot description, xacro)
@@ -65,5 +65,8 @@
     <parent link="world"/>
     <child link="base_link"/>
-    <origin xyz="0.0 0.0 1.54" rpy="1.5707 0.0 1.5707"/>
+    <origin xyz="0.0 0.0 1.54" rpy="0.0 1.5707 0.0"/>
+            <!-- was this before sliding base added
+            <origin xyz="0.0 0.0 1.54" rpy="1.5707 0.0 1.5707"/>
+            -->
   </joint>
   <link name="tool0_controller"/>
